Commit message: Added compatibilty for camera bracket

File: triple_s_util/urdf/ur5.urdf.xacro (robot description, xacro)
@@ -11,4 +11,29 @@
         <xacro:include filename="$(find ur_description)/urdf/ur5_robot.urdf.xacro"/>
     </xacro:unless>
+    <!-- Camera Bracket-->
+    <link name="Camera_bracket">
+        <inertial>
+            <origin rpy="0 0 0" xyz="0 0.01 -0.2239"/>
+            <mass value="0.00995"/>
+            <inertia ixx="25.39883" ixy="0.0" ixz="0.0" iyy="31.75919" iyz="-0.4794" izz="6.41732"/>
+        </inertial>
+        <visual>
+            <origin xyz="0.0 0.0 0.0" rpy="0.0 0.0 0.0"/>
+            <geometry>
+                <mesh filename="package://triple_s_util/meshes/Camera_bracket.STL" scale="0.001 0.001 0.001"/>
+            </geometry>
+        </visual>
+        <collision>
+            <origin xyz="0.0 0.0 0.0" rpy="0.0 0.0 0.0"/>
+            <geometry>
+                <mesh filename="package://triple_s_util/meshes/Camera_bracket.STL" scale="0.001 0.001 0.001"/>
+            </geometry>
+        </collision>
+    </link>
+    <joint name="bracket_ur5" type="fixed">
+        <parent link="ee_link" />
+        <child link="Camera_bracket" />
+        <origin xyz="0 -0.0305 0.06298" rpy="${pi} 0 ${pi/2}" />
+    </joint>
     <!-- Gripper -->
     <xacro:property name="gripper_name" value="$(arg gripper_name)" />
@@ -19,5 +44,5 @@
             <parent link="ee_link" />
             <child link="rg2_base_link" />
-            <origin xyz="0 0 0" rpy="0 0 0" />
+            <origin xyz="0.002 0 0" rpy="0 0 0" />
         </joint>
     </xacro:if>
@@ -28,5 +53,5 @@
             <parent link="ee_link" />
             <child link="robotiq_arg2f_base_link" />
-            <origin xyz="0 0 0" rpy="0 ${pi/2} 0" />
+            <origin xyz="0.002 0 0" rpy="0 ${pi/2} 0" />
         </joint>
     </xacro:if>
@@ -39,6 +64,6 @@
     </xacro:unless>
     <xacro:if value="$(arg camera_on_robot)">
-        <xacro:camerasim parent="wrist_2_link">
-            <origin xyz="0 0.035 0.134" rpy="0 0 ${pi/2}"/>
+        <xacro:camerasim parent="Camera_bracket">
+            <origin xyz="0.03 0.012 0" rpy="0 0 ${pi/2}"/>
         </xacro:camerasim>
     </xacro:if>

Commit message: Remove table world, and add collission aware table

File: triple_s_util/urdf/ur5.urdf.xacro (robot description, xacro)
@@ -4,11 +4,33 @@
     <xacro:arg name="camera_on_robot" default="false"/>
     <xacro:arg name="gripper_name" default="robotiq"/>
+    <xacro:arg name="transmission_hw_interface" default="hardware_interface/PositionJointInterface"/>
+    <xacro:arg name="kinematics_config" default="$(find ur_description)/config/ur5_default.yaml"/>
+    <link name="world"/>
     <!-- UR5 -->
+    <xacro:include filename="$(find ur_description)/urdf/common.gazebo.xacro" />
+    <xacro:include filename="$(find ur_description)/urdf/ur5.urdf.xacro" />
     <xacro:if value="$(arg limited)">
-        <xacro:include filename="$(find ur_description)/urdf/ur5_joint_limited_robot.urdf.xacro" />
+        <xacro:ur5_robot prefix="" joint_limited="true"
+            shoulder_pan_lower_limit="${-pi}" shoulder_pan_upper_limit="${pi}"
+            shoulder_lift_lower_limit="${-pi}" shoulder_lift_upper_limit="${pi}"
+            elbow_joint_lower_limit="${-pi}" elbow_joint_upper_limit="${pi}"
+            wrist_1_lower_limit="${-pi}" wrist_1_upper_limit="${pi}"
+            wrist_2_lower_limit="${-pi}" wrist_2_upper_limit="${pi}"
+            wrist_3_lower_limit="${-pi}" wrist_3_upper_limit="${pi}"
+            transmission_hw_interface="$(arg transmission_hw_interface)"
+            kinematics_file="${load_yaml('$(arg kinematics_config)')}"
+        />
     </xacro:if>
     <xacro:unless value="$(arg limited)">
-        <xacro:include filename="$(find ur_description)/urdf/ur5_robot.urdf.xacro"/>
+        <xacro:ur5_robot prefix="" joint_limited="false"
+            transmission_hw_interface="$(arg transmission_hw_interface)"
+            kinematics_file="${load_yaml('$(arg kinematics_config)')}"
+        />
     </xacro:unless>
+    <joint name="ur5_world_joint" type="fixed">
+        <parent link="world"/>
+        <child link="base_link"/>
+        <origin xyz="0 0 1" rpy="0 0 0"/>
+    </joint>
     <!-- Camera Bracket-->
     <link name="Camera_bracket">
@@ -69,5 +91,5 @@
     </xacro:if>
     <!-- environment -->
-    <xacro:include filename="$(find triple_s_util)/urdf/environment.urdf.xacro" />
+    <xacro:include filename="$(find triple_s_util)/urdf/saxion_table.urdf.xacro" />
     <xacro:environment parent="world" />
 </robot>

Commit message: Add Viro table, remove dependencies

File: triple_s_util/urdf/ur5.urdf.xacro (robot description, xacro)
@@ -6,4 +6,5 @@
     <xacro:arg name="transmission_hw_interface" default="hardware_interface/PositionJointInterface"/>
     <xacro:arg name="kinematics_config" default="$(find ur_description)/config/ur5_default.yaml"/>
+    <xacro:arg name="environment" default="viro" />
     <link name="world"/>
     <!-- UR5 -->
@@ -28,9 +29,24 @@
         />
     </xacro:unless>
-    <joint name="ur5_world_joint" type="fixed">
-        <parent link="world"/>
-        <child link="base_link"/>
-        <origin xyz="0 0 1" rpy="0 0 0"/>
-    </joint>
+    <!-- environment -->
+    <xacro:property name="environment_name" value="$(arg environment)"/>
+    <xacro:if value="${environment_name == 'saxion'}">
+        <xacro:include filename="$(find triple_s_util)/urdf/saxion_table.urdf.xacro" />
+        <xacro:environment parent="world" />
+        <joint name="ur5_world_joint" type="fixed">
+            <parent link="world"/>
+            <child link="base_link"/>
+            <origin xyz="0 0.1 1" rpy="0 0 0"/>
+        </joint>
+    </xacro:if>
+    <xacro:if value="${environment_name == 'viro'}">
+        <xacro:include filename="$(find triple_s_util)/urdf/viro_table.urdf.xacro" />
+        <xacro:environment parent="world" />
+        <joint name="ur5_world_joint" type="fixed">
+            <parent link="world"/>
+            <child link="base_link"/>
+            <origin xyz="0 0 0.759" rpy="0 0 0"/>
+        </joint>
+    </xacro:if>
     <!-- Camera Bracket-->
     <link name="Camera_bracket">
@@ -90,6 +106,3 @@
         </xacro:camerasim>
     </xacro:if>
-    <!-- environment -->
-    <xacro:include filename="$(find triple_s_util)/urdf/saxion_table.urdf.xacro" />
-    <xacro:environment parent="world" />
 </robot>
