Commit message: Update viro table

File: triple_s_util/urdf/viro_table.urdf.xacro (robot description, xacro)
@@ -11,14 +11,11 @@
                 <origin xyz="0 0 0" rpy="0 0 0"/>
                 <geometry>
-                    <mesh filename="package://triple_s_util/meshes/viro/table.dae"/>
+                    <mesh filename="package://triple_s_util/meshes/viro/viro_table.dae"/>
                 </geometry>
-                <material name="green">
-                    <color rgba="0 0.61 0.51 1.0"/>
-                </material>
             </visual>
             <collision>
                 <origin xyz="0 0 0" rpy="0 0 0"/>
                 <geometry>
-                    <mesh filename="package://triple_s_util/meshes/viro/table.STL"/>
+                    <mesh filename="package://triple_s_util/meshes/viro/viro_table.stl"/>
                 </geometry>
             </collision>
@@ -27,5 +24,5 @@
             <parent link="${parent}" />
             <child link="${prefix}table" />
-            <origin xyz="0 0 0" rpy="0 0 ${pi/2}" />
+            <origin xyz="0 0 0.05" rpy="0 0 ${pi}" />
         </joint>
     </xacro:macro>
