Commit message: Cleanup unused meshes

File: triple_s_util/urdf/saxion_table.urdf.xacro (robot description, xacro)
@@ -11,5 +11,5 @@
                 <origin xyz="0 0 0" rpy="0 0 0"/>
                 <geometry>
-                    <mesh filename="package://triple_s_util/meshes/saxion_table.dae"/>
+                    <mesh filename="package://triple_s_util/meshes/saxion/saxion_table.dae"/>
                 </geometry>
                 <material name="green">
@@ -20,5 +20,5 @@
                 <origin xyz="0 0 0" rpy="0 0 0"/>
                 <geometry>
-                    <mesh filename="package://triple_s_util/meshes/saxion_table.dae"/>
+                    <mesh filename="package://triple_s_util/meshes/saxion/saxion_table.dae"/>
                 </geometry>
             </collision>

File: triple_s_util/urdf/ur5.urdf.xacro (robot description, xacro)
@@ -59,5 +59,5 @@
             <origin xyz="0.0 0.0 0.0" rpy="0.0 0.0 0.0"/>
             <geometry>
-                <mesh filename="package://triple_s_util/meshes/Camera_bracket.STL" scale="0.001 0.001 0.001"/>
+                <mesh filename="package://triple_s_util/meshes/camera_bracket.stl" scale="0.001 0.001 0.001"/>
             </geometry>
         </visual>
@@ -65,5 +65,5 @@
             <origin xyz="0.0 0.0 0.0" rpy="0.0 0.0 0.0"/>
             <geometry>
-                <mesh filename="package://triple_s_util/meshes/Camera_bracket.STL" scale="0.001 0.001 0.001"/>
+                <mesh filename="package://triple_s_util/meshes/camera_bracket.stl" scale="0.001 0.001 0.001"/>
             </geometry>
         </collision>
