Commit message: Add configurable poses file and update docs

File: triple_s_util/config/ur5_gripper.srdf.xacro (robot description, xacro)
@@ -2,4 +2,5 @@
 <robot name="ur5" xmlns:xacro="http://www.ros.org/wiki/xacro">
     <xacro:arg name="gripper" default="robotiq" />
+    <xacro:arg name="poses" default="$(find triple_s_util)/config/poses/test_sim.srdf"/>
     <xacro:property name="gripper" value="$(arg gripper)" />
     <xacro:include filename="$(find ur5_moveit_config)/config/ur5.srdf" />
@@ -14,12 +15,4 @@
     </xacro:if>
     <disable_collisions link1="Camera_bracket" link2="wrist_3_link"/>
-    <group_state name="home_pose" group="manipulator">
-        <joint name="elbow_joint" value="1.5707" />
-        <joint name="shoulder_lift_joint" value="-1.5707" />
-        <joint name="shoulder_pan_joint" value="0" />
-        <joint name="wrist_1_joint" value="-1.5707" />
-        <joint name="wrist_2_joint" value="-1.5707" />
-        <joint name="wrist_3_joint" value="0" />
-    </group_state>
-    <xacro:include filename="$(find triple_s_util)/config/poses.srdf" />
+    <xacro:include filename="$(arg poses)" />
 </robot>

Commit message: Rotate camera

File: triple_s_util/config/ur5_gripper.srdf.xacro (robot description, xacro)
@@ -6,13 +6,14 @@
     <xacro:include filename="$(find ur5_moveit_config)/config/ur5.srdf" />
     <xacro:if value="${gripper == 'rg2'}">
-        <xacro:include filename="$(find onrobot_rg2)/urdf/rg2.srdf"/>
-        <disable_collisions link1="Camera_bracket" link2="rg2_base_link"/>
+        <xacro:include filename="$(find onrobot_rg2)/urdf/rg2.srdf" />
+        <disable_collisions link1="camera_bracket" link2="rg2_base_link" />
     </xacro:if>
     <xacro:if value="${gripper == 'robotiq'}">
-        <xacro:include filename="$(find robotiq_2f_85_gripper_visualization)/config/robotiq_2f_85.srdf"/>
-        <disable_collisions link1="Camera_bracket" link2="robotiq_arg2f_base_link"/>
-        <disable_collisions link1="robotiq_arg2f_base_link" link2="wrist_3_link" reason="Adjacent"/>
+        <xacro:include filename="$(find robotiq_2f_85_gripper_visualization)/config/robotiq_2f_85.srdf" />
+        <disable_collisions link1="camera_bracket" link2="robotiq_arg2f_base_link" />
+        <disable_collisions link1="robotiq_arg2f_base_link" link2="wrist_3_link" reason="Adjacent" />
     </xacro:if>
-    <disable_collisions link1="Camera_bracket" link2="wrist_3_link"/>
+    <disable_collisions link1="camera_bracket" link2="wrist_3_link" />
+    <disable_collisions link1="base_link" link2="environment_table" />
     <xacro:include filename="$(arg poses)" />
 </robot>

File: triple_s_util/urdf/ur5.urdf.xacro (robot description, xacro)
@@ -50,5 +50,5 @@
     </xacro:if>
     <!-- Camera Bracket-->
-    <link name="Camera_bracket">
+    <link name="camera_bracket">
         <inertial>
             <origin rpy="0 0 0" xyz="0 0.01 -0.2239"/>
@@ -71,5 +71,5 @@
     <joint name="bracket_ur5" type="fixed">
         <parent link="ee_link" />
-        <child link="Camera_bracket" />
+        <child link="camera_bracket" />
         <origin xyz="0 -0.0305 0.06298" rpy="${pi} 0 ${pi/2}" />
     </joint>
@@ -102,6 +102,6 @@
     </xacro:unless>
     <xacro:if value="$(arg camera_on_robot)">
-        <xacro:camerasim parent="Camera_bracket">
-            <origin xyz="0.03 0.012 0" rpy="0 0 ${pi/2}"/>
+        <xacro:camerasim parent="camera_bracket">
+            <origin xyz="0.03 0.012 0.025" rpy="${pi} 0 ${pi/2}"/>
         </xacro:camerasim>
     </xacro:if>

Commit message: Move planning point location

File: triple_s_util/config/ur5_gripper.srdf.xacro (robot description, xacro)
@@ -4,8 +4,16 @@
     <xacro:arg name="poses" default="$(find triple_s_util)/config/poses/test_sim.srdf"/>
     <xacro:property name="gripper" value="$(arg gripper)" />
-    <xacro:include filename="$(find ur5_moveit_config)/config/ur5.srdf" />
+    <xacro:include filename="$(find triple_s_util)/config/ur5.srdf" />
     <xacro:if value="${gripper == 'rg2'}">
         <xacro:include filename="$(find onrobot_rg2)/urdf/rg2.srdf" />
         <disable_collisions link1="camera_bracket" link2="rg2_base_link" />
+        <!-- Passive joints cannot be used for planning -->
+        <passive_joint name="rg2_base_link" />
+        <passive_joint name="rg2_left_finger" />
+        <passive_joint name="rg2_right_finger" />
+        <passive_joint name="rg2_right_outer_link" />
+        <passive_joint name="rg2_left_outer_link" />
+        <passive_joint name="rg2_left_inner_link" />
+        <passive_joint name="rg2_right_inner_link" />
     </xacro:if>
     <xacro:if value="${gripper == 'robotiq'}">

File: triple_s_util/urdf/ur5.urdf.xacro (robot description, xacro)
@@ -75,12 +75,21 @@
     </joint>
     <!-- Gripper -->
+    <!-- The following link must be placed on the gripping location on the gripper (between the two fingers)-->
+    <link name="gripper_sim_link"/>
     <xacro:property name="gripper_name" value="$(arg gripper_name)" />
     <xacro:if value="${gripper_name == 'rg2'}">
         <xacro:include filename="$(find onrobot_rg2)/urdf/rg2.macro.xacro" />
         <xacro:onrobot_rg2 prefix="rg2_" standalone="false"/>
+        <!-- Link the rg2 to the ur5-->
         <joint name="ur5_gripper_link" type="fixed">
             <parent link="ee_link" />
             <child link="rg2_base_link" />
             <origin xyz="0.002 0 0" rpy="0 0 0" />
+        </joint>
+        <!-- Define the gripping location-->
+        <joint name="gripper_sim_link_joint" type="fixed">
+            <parent link="ee_link"/>
+            <child link="gripper_sim_link" />
+            <origin xyz="0.17 0 0" rpy="0 0 0"/>
         </joint>
     </xacro:if>
